Commit message: extract dimensions properties

File: ros2_ws/src/robot_description/description/arm.urdf.xacro (robot description, xacro)
@@ -1,4 +1,5 @@
 <?xml version="1.0"?>
 <robot xmlns:xacro="http://www.ros.org/wiki/xacro" name="arm">
+    <xacro:include filename="dimensions.xacro"/>
     <link name="world"/>
     <joint name="base_joint" type="fixed">
@@ -7,7 +8,4 @@
         <origin xyz="0.0 0.0 0.0" rpy="0.0 0.0 0.0"/>
     </joint>
-    <xacro:property name="base_length" value="2.5"/>
-    <xacro:property name="base_width" value="1.5"/>
-`    <xacro:property name="base_height" value=".1"/>
     <link name="base_link">
         <visual>
@@ -28,21 +26,18 @@
         <child link="link1"/>
         <axis xyz="0 0 1"/>
-        <limit lower="-3.14159" upper="3.14159" velocity="50.0" effort="1000.0"/>
+        <limit lower="${axis1_lower}" upper="${axis1_upper}" velocity="50.0" effort="1000.0"/>
         <origin xyz="0 0 0" rpy="0 0 0"/>
     </joint>
-    <xacro:property name="link1_length" value="0.5"/>
-    <xacro:property name="link1_width" value="0.25"/>
-    <xacro:property name="link1_height" value="0.15"/>
     <link name="link1">
         <visual>
-            <origin xyz="0.0 0.0 ${base_height + (link1_height / 2)}" rpy="0.0 0.0 0.0"/>
+            <origin xyz="0.0 0.0 ${link1_length/2}" rpy="0.0 0.0 0.0"/>
             <geometry>
-                <cylinder radius="${link1_width}" length="${link1_height}"/>
+                <cylinder radius="${link1_radius}" length="${link1_length}"/>
             </geometry>
         </visual>
         <collision>
-            <origin xyz="0.0 0.0 ${link1_length / 2}" rpy="0.0 0.0 0.0"/>
+            <origin xyz="0.0 0.0 ${link1_length/2}" rpy="0.0 0.0 0.0"/>
             <geometry>
-                <cylinder radius="${link1_width}" length="${link1_height}"/>
+                <cylinder radius="${link1_radius}" length="${link1_length}"/>
             </geometry>
         </collision>
@@ -52,10 +47,7 @@
         <child link="link2"/>
         <axis xyz="0 1 0"/>
-        <limit lower="-3.14159" upper="3.14159" velocity="50.0" effort="1000.0"/>
-        <origin xyz="0 0 ${base_height + link1_height}" rpy="0 0 0"/>
+        <limit lower="${axis2_lower}" upper="${axis2_upper}" velocity="50.0" effort="1000.0"/>
+        <origin xyz="0 0 ${base_height + link1_length}" rpy="0 0 0"/>
     </joint>
-    <xacro:property name="link2_length" value="1"/>
-    <xacro:property name="link2_width" value="0.25"/>
-    <xacro:property name="link2_height" value="0.25"/>
     <link name="link2">
         <visual>
@@ -76,10 +68,7 @@
         <child link="link3"/>
         <axis xyz="0 1 0"/>
-        <limit lower="-3.14159" upper="3.14159" velocity="50.0" effort="1000.0"/>
+        <limit lower="${axis3_lower}" upper="${axis3_upper}" velocity="50.0" effort="1000.0"/>
         <origin xyz="0 0 ${link2_length}" rpy="0 0 0"/>
     </joint>
-    <xacro:property name="link3_length" value="1"/>
-    <xacro:property name="link3_width" value="0.25"/>
-    <xacro:property name="link3_height" value="0.25"/>
     <link name="link3">
         <visual>
@@ -100,10 +89,7 @@
         <child link="link4"/>
         <axis xyz="0 1 0"/>
-        <limit lower="-3.14159" upper="3.14159" velocity="50.0" effort="1000.0"/>
+        <limit lower="${axis4_lower}" upper="${axis4_upper}" velocity="50.0" effort="1000.0"/>
         <origin xyz="0 0 ${link3_length}" rpy="0 0 0"/>
     </joint>
-    <xacro:property name="link4_length" value="0.25"/>
-    <xacro:property name="link4_width" value="0.25"/>
-    <xacro:property name="link4_height" value="0.25"/>
     <link name="link4">
         <visual>
@@ -124,10 +110,7 @@
         <child link="link5"/>
         <axis xyz="0 0 1"/>
-        <limit lower="-3.14159" upper="3.14159" velocity="50.0" effort="1000.0"/>
+        <limit lower="${axis5_lower}" upper="${axis5_upper}" velocity="50.0" effort="1000.0"/>
         <origin xyz="0 0 ${link4_length}" rpy="0 0 0"/>
     </joint>
-    <xacro:property name="link5_length" value="0.25"/>
-    <xacro:property name="link5_width" value="0.25"/>
-    <xacro:property name="link5_height" value="0.25"/>
     <link name="link5">
         <visual>
