Commit message: add materials

File: ros2_ws/src/robot_description/description/arm/arm.urdf.xacro (robot description, xacro)
@@ -2,4 +2,5 @@
 <robot xmlns:xacro="http://www.ros.org/wiki/xacro" name="arm">
     <xacro:include filename="dimensions.xacro"/>
+    <xacro:include filename="../materials.xacro"/>
     <link name="world"/>
     <joint name="base_joint" type="fixed">
@@ -14,4 +15,5 @@
                 <box size="${base_length} ${base_width} ${base_height}"/>
             </geometry>
+            <material name="blue"></material>
         </visual>
         <collision>
@@ -35,4 +37,5 @@
                 <cylinder radius="${link1_radius}" length="${link1_length}"/>
             </geometry>
+            <material name="orange"></material>
         </visual>
         <collision>
@@ -56,4 +59,5 @@
                 <box size="${link2_length} ${link2_width} ${link2_height}"/>
             </geometry>
+            <material name="green"></material>
         </visual>
         <collision>
@@ -77,4 +81,5 @@
                 <box size="${link3_length} ${link3_width} ${link3_height}"/>
             </geometry>
+            <material name="magenta"></material>
         </visual>
         <collision>
@@ -98,4 +103,5 @@
                 <box size="${link4_length} ${link4_width} ${link4_height}"/>
             </geometry>
+            <material name="cyan"></material>
         </visual>
         <collision>
@@ -119,4 +125,5 @@
                 <box size="${link5_length} ${link5_width} ${link5_height}"/>
             </geometry>
+            <material name="white"></material>
         </visual>
         <collision>

Commit message: not showing in gazebo

File: ros2_ws/src/robot_description/description/arm/arm.urdf.xacro (robot description, xacro)
@@ -3,5 +3,6 @@
     <xacro:include filename="dimensions.xacro"/>
     <xacro:include filename="../materials.xacro"/>
-    <link name="world"/>
+    <xacro:include filename="../inertias.xacro"/>
+    <link name="world"></link>
     <joint name="base_joint" type="fixed">
         <parent link="world"/>
@@ -23,4 +24,7 @@
             </geometry>
         </collision>
+        <xacro:inertial_box mass="1" length="0" width="0" height="0">
+            <origin xyz="0.0 0.0 0.0" rpy="0.0 0.0 0.0"/>
+        </xacro:inertial_box>
     </link>
     <joint name="axis1" type="revolute">
@@ -30,4 +34,5 @@
         <limit lower="${axis1_lower}" upper="${axis1_upper}" velocity="50.0" effort="1000.0"/>
         <origin xyz="0 0 0" rpy="0 0 0"/>
+        <dynamics damping="10.0" friction="10.0"/>
     </joint>
     <link name="link1">
@@ -45,4 +50,7 @@
             </geometry>
         </collision>
+        <xacro:inertial_cylinder mass="1" length="${link1_length}" radius="${link1_radius}">
+            <origin xyz="${link1_length/2} 0.0 0.0" rpy="0.0 0.0 0.0"/>
+        </xacro:inertial_cylinder>
     </link>
     <joint name="axis2" type="revolute">
@@ -52,4 +60,5 @@
         <limit lower="${axis2_lower}" upper="${axis2_upper}" velocity="50.0" effort="1000.0"/>
         <origin xyz="0 0 ${base_height + link1_length}" rpy="0 0 0"/>
+        <dynamics damping="10.0" friction="10.0"/>
     </joint>
     <link name="link2">
@@ -67,4 +76,7 @@
             </geometry>
         </collision>
+        <xacro:inertial_box mass="1" length="${link2_length}" width="${link2_width}" height="${link2_height}">
+            <origin xyz="${link2_length/2} 0.0 0.0" rpy="0.0 0.0 0.0"/>
+        </xacro:inertial_box>
     </link>
     <joint name="axis3" type="revolute">
@@ -74,4 +86,5 @@
         <limit lower="${axis3_lower}" upper="${axis3_upper}" velocity="50.0" effort="1000.0"/>
         <origin xyz="0 0 ${link2_length}" rpy="0 0 0"/>
+        <dynamics damping="10.0" friction="10.0"/>
     </joint>
     <link name="link3">
@@ -89,4 +102,7 @@
             </geometry>
         </collision>
+        <xacro:inertial_box mass="1" length="${link3_length}" width="${link3_width}" height="${link3_width}">
+            <origin xyz="${link3_length} 0.0 0.0" rpy="0.0 0.0 0.0"/>
+        </xacro:inertial_box>
     </link>
     <joint name="axis4" type="revolute">
@@ -96,4 +112,5 @@
         <limit lower="${axis4_lower}" upper="${axis4_upper}" velocity="50.0" effort="1000.0"/>
         <origin xyz="0 0 ${link3_length}" rpy="0 0 0"/>
+        <dynamics damping="10.0" friction="10.0"/>
     </joint>
     <link name="link4">
@@ -111,4 +128,7 @@
             </geometry>
         </collision>
+        <xacro:inertial_box mass="1" length="${link4_length}" width="${link4_width}" height="${link4_width}">
+            <origin xyz="${link4_length} 0.0 0.0" rpy="0.0 0.0 0.0"/>
+        </xacro:inertial_box>
     </link>
     <joint name="axis5" type="revolute">
@@ -118,4 +138,5 @@
         <limit lower="${axis5_lower}" upper="${axis5_upper}" velocity="50.0" effort="1000.0"/>
         <origin xyz="0 0 ${link4_length}" rpy="0 0 0"/>
+        <dynamics damping="10.0" friction="10.0"/>
     </joint>
     <link name="link5">
@@ -133,4 +154,7 @@
             </geometry>
         </collision>
+        <xacro:inertial_box mass="1" length="${link5_length}" width="${link5_width}" height="${link5_width}">
+            <origin xyz="${link5_length} 0.0 0.0" rpy="0.0 0.0 0.0"/>
+        </xacro:inertial_box>
     </link>
 </robot>
