Commit message: fix typo in world chassis

File: ros2_ws/src/turtlebot/description/robot_core.xacro (robot description, xacro)
@@ -5,11 +5,11 @@
     <!-- BASE -->
     <link name="base_link"/>
-    <!-- CHASIS -->
+    <!-- chassis -->
     <joint name="chasis_joint" type="fixed">
         <parent link="base_link"/>
-        <child link="chasis"/>
+        <child link="chassis"/>
         <origin xyz="-0.1 0.0 0.0" rpy="0.0 0.0 0.0"/>
     </joint>
-    <link name="chasis">
+    <link name="chassis">
         <visual>
             <material name="white"></material>
@@ -77,5 +77,5 @@
     <!-- CASTER WHEEL -->
     <joint name="caster_wheel_joint" type="fixed">
-        <parent link="chasis"/>
+        <parent link="chassis"/>
         <child link="caster_wheel"/>
         <origin xyz="0.24 0.0 0.0" rpy="0.0 0.0 0.0"/>
